Commit message: Try to get the robot showing in gazebo

File: robot_challenge_description/src/description/robot_challenge_description.urdf (robot description, URDF)
Before this commit: robot ackermann_steering_vehicle, 9 links, 8 joints
Links:
- added link imu_link; collision box size=0.1 0.1 0.1; visual box size=0.1 0.1 0.1
- link base_link: mass ${body_mass} -> None
- link front_left_steering_link: mass 0.01 -> None
- link front_right_steering_link: mass 0.01 -> None
Joints:
- added joint imu_joint: type fixed, parent camera_link, child imu_link, origin xyz=0 0 0.01

Commit message: Some updates to get teh bot loading more correctly

File: robot_challenge_description/src/description/robot_challenge_description.urdf (robot description, URDF)
Before this commit: robot ackermann_steering_vehicle, 10 links, 9 joints
Links:
- link front_left_steering_link: mass None -> 0.01
- link front_right_steering_link: mass None -> 0.01

Commit message: Fix joint_state_publisher

File: robot_challenge_description/src/description/robot_challenge_description.urdf (robot description, URDF)
Before this commit: robot ackermann_steering_vehicle, 10 links, 9 joints
Links:
- link base_link: geometry collision box size=2.0 1.0 0.5; visual box size=2.0 1.0 0.5
- link camera_link: geometry collision box size=0.1 0.1 0.1; visual box size=0.1 0.1 0.1
- link camera_stick_link: geometry collision box size=0.2 0.2 1.5; visual box size=0.2 0.2 1.5
- link front_left_wheel_link: mass ${wheel_mass} -> 28.27433385; geometry collision cylinder length=0.1 radius=0.3; visual cylinder length=0.1 radius=0.3
- link front_right_wheel_link: mass ${wheel_mass} -> 28.27433385; geometry collision cylinder length=0.1 radius=0.3; visual cylinder length=0.1 radius=0.3
- link rear_left_wheel_link: geometry collision cylinder length=0.1 radius=0.3; visual cylinder length=0.1 radius=0.3
- link rear_right_wheel_link: geometry collision cylinder length=0.1 radius=0.3; visual cylinder length=0.1 radius=0.3
Joints:
- joint camera_joint: origin xyz=0.0 ${-camera_box_size/2 - camera_stick_size/2} ${camera_height/2} rpy=0 ${camera_pitch} 0 -> xyz=0.0 -0.15000000000000002 0.75 rpy=0 0.1 0
- joint camera_stick_joint: origin xyz=${body_length/2 - camera_stick_size/2} ${camera_box_size/2 + camera_stick_size/2} ${camera_height/2} rpy=0.0 0.0 0.0 -> xyz=0.9 0.15000000000000002 0.75 rpy=0.0 0.0 0.0
- joint front_left_steering_joint: limit lower=${-max_steering_angle} upper=${max_steering_angle} effort=${max_steering_effort} velocity=${max_steering_angular_velocity} -> lower=-0.6108 upper=0.6108 effort=1.0 velocity=1.570796; origin xyz=${wheel_offset} ${wheel_separation/2} -${wheel_radius/2} rpy=0 0 0 -> xyz=0.7 0.55 -0.15 rpy=0 0 0
- joint front_left_wheel_joint: limit effort=${max_effort} velocity=${max_wheel_angular_velocity} -> effort=10.0 velocity=3.3333333333333335
- joint front_right_steering_joint: limit lower=${-max_steering_angle} upper=${max_steering_angle} effort=${max_steering_effort} velocity=${max_steering_angular_velocity} -> lower=-0.6108 upper=0.6108 effort=1.0 velocity=1.570796; origin xyz=${wheel_offset} ${-wheel_separation/2} -${wheel_radius/2} rpy=0 0 0 -> xyz=0.7 -0.55 -0.15 rpy=0 0 0
- joint front_right_wheel_joint: limit effort=${max_effort} velocity=${max_wheel_angular_velocity} -> effort=10.0 velocity=3.3333333333333335
- joint rear_left_wheel_joint: limit effort=${max_effort} velocity=${max_wheel_angular_velocity} -> effort=10.0 velocity=3.3333333333333335; origin xyz=-${wheel_offset} ${wheel_separation/2} -${wheel_radius/2} rpy=0 0 0 -> xyz=-0.7 0.55 -0.15 rpy=0 0 0
- joint rear_right_wheel_joint: limit effort=${max_effort} velocity=${max_wheel_angular_velocity} -> effort=10.0 velocity=3.3333333333333335; origin xyz=-${wheel_offset} ${-wheel_separation/2} -${wheel_radius/2} rpy=0 0 0 -> xyz=-0.7 -0.55 -0.15 rpy=0 0 0

Commit message: Resize bot and add build script

File: robot_challenge_description/src/description/robot_challenge_description.urdf (robot description, URDF)
Before this commit: robot ackermann_steering_vehicle, 10 links, 9 joints
Links:
- link base_link: geometry collision box size=0.557 0.249 0.241; visual box size=0.557 0.249 0.241
- link camera_link: geometry collision box size=0.01 0.01 0.01; visual box size=0.01 0.01 0.01
- link camera_stick_link: geometry collision box size=0.01 0.01 0.01; visual box size=0.01 0.01 0.01
- link front_left_wheel_link: mass 28.27433385 -> 0.52841588373; geometry collision cylinder length=0.05 radius=0.058; visual cylinder length=0.05 radius=0.058
- link front_right_wheel_link: mass 28.27433385 -> 0.52841588373; geometry collision cylinder length=0.05 radius=0.058; visual cylinder length=0.05 radius=0.058
- link rear_left_wheel_link: geometry collision cylinder length=0.05 radius=0.058; visual cylinder length=0.05 radius=0.058
- link rear_right_wheel_link: geometry collision cylinder length=0.05 radius=0.058; visual cylinder length=0.05 radius=0.058
Joints:
- joint camera_joint: origin xyz=0.0 -0.15000000000000002 0.75 rpy=0 0.1 0 -> xyz=0.0 -0.01 0.005 rpy=0 0.1 0
- joint camera_stick_joint: origin xyz=0.9 0.15000000000000002 0.75 rpy=0.0 0.0 0.0 -> xyz=0.2735 0.01 0.005 rpy=0.0 0.0 0.0
- joint front_left_steering_joint: origin xyz=0.7 0.55 -0.15 rpy=0 0 0 -> xyz=0.22050000000000003 0.1495 -0.029 rpy=0 0 0
- joint front_left_wheel_joint: limit effort=10.0 velocity=3.3333333333333335 -> effort=10.0 velocity=17.241379310344826
- joint front_right_steering_joint: origin xyz=0.7 -0.55 -0.15 rpy=0 0 0 -> xyz=0.22050000000000003 -0.1495 -0.029 rpy=0 0 0
- joint front_right_wheel_joint: limit effort=10.0 velocity=3.3333333333333335 -> effort=10.0 velocity=17.241379310344826
- joint rear_left_wheel_joint: limit effort=10.0 velocity=3.3333333333333335 -> effort=10.0 velocity=17.241379310344826; origin xyz=-0.7 0.55 -0.15 rpy=0 0 0 -> xyz=-0.22050000000000003 0.1495 -0.029 rpy=0 0 0
- joint rear_right_wheel_joint: limit effort=10.0 velocity=3.3333333333333335 -> effort=10.0 velocity=17.241379310344826; origin xyz=-0.7 -0.55 -0.15 rpy=0 0 0 -> xyz=-0.22050000000000003 -0.1495 -0.029 rpy=0 0 0

File: robot_challenge_description/src/description/robot_challenge_description.xacro (robot description, xacro)
@@ -6,10 +6,10 @@
   -->
   <!-- Arguments -->
-  <xacro:arg name="body_length" default="2.0" />
-  <xacro:arg name="body_width" default="1.0" />
-  <xacro:arg name="body_height" default="0.5" />
+  <xacro:arg name="body_length" default=".557" />
+  <xacro:arg name="body_width" default=".249" />
+  <xacro:arg name="body_height" default="0.241" />
   <xacro:arg name="body_density" default="1000.0" />
-  <xacro:arg name="wheel_radius" default="0.3" />
-  <xacro:arg name="wheel_width" default="0.1" />
+  <xacro:arg name="wheel_radius" default="0.058" />
+  <xacro:arg name="wheel_width" default="0.05" />
   <xacro:arg name="wheel_density" default="1000.0" />
   <xacro:arg name="max_steering_angle" default="0.6108" />
@@ -18,7 +18,7 @@
   <xacro:arg name="max_velocity" default="1.0" />
   <xacro:arg name="max_effort" default="10.0" />
-  <xacro:arg name="camera_box_size" default="0.1" />
-  <xacro:arg name="camera_stick_size" default="0.2" />
-  <xacro:arg name="camera_height" default="1.5" />
+  <xacro:arg name="camera_box_size" default="0.01" />
+  <xacro:arg name="camera_stick_size" default="0.01" />
+  <xacro:arg name="camera_height" default=".01" />
   <xacro:arg name="camera_pitch" default="0.1" />
   <xacro:arg name="camera_fov" default="1.570796" />

Commit message: Add lidar and move camera

File: robot_challenge_description/src/description/robot_challenge_description.urdf (robot description, URDF)
Before this commit: robot ackermann_steering_vehicle, 10 links, 9 joints
Links:
- added link lidar_link; collision cylinder length=0.0528 radius=0.0325; visual cylinder length=0.0528 radius=0.0325
- added link steering_wheel_link
- link base_link: geometry collision box size=0.474 0.192 0.138; visual box size=0.474 0.192 0.138
- link camera_link: geometry collision box size=0.0254 0.1 0.0254; visual box size=0.0254 0.1 0.0254
- link camera_stick_link: geometry collision box size=0.01 0.01 0.0254; visual box size=0.01 0.01 0.0254
- link front_left_wheel_link: mass 0.52841588373 -> 0.70630856753625; geometry collision cylinder length=0.068 radius=0.0575; visual cylinder length=0.068 radius=0.0575
- link front_right_wheel_link: mass 0.52841588373 -> 0.70630856753625; geometry collision cylinder length=0.068 radius=0.0575; visual cylinder length=0.068 radius=0.0575
- link imu_link: geometry collision box size=0.0254 0.1 0.0254; visual box size=0.0254 0.1 0.0254
- link rear_left_wheel_link: geometry collision cylinder length=0.068 radius=0.0575; visual cylinder length=0.068 radius=0.0575
- link rear_right_wheel_link: geometry collision cylinder length=0.068 radius=0.0575; visual cylinder length=0.068 radius=0.0575
Joints:
- added joint lidar_joint: type fixed, parent base_link, child lidar_link, origin xyz=0.22199999999999998 0 0.042600000000000006 rpy=0.0 0.0 0.0, axis 0 1 0
- added joint steering_wheel_joint: type continuous, parent base_link, child steering_wheel_link, origin xyz=0 0 0.0
- joint camera_joint: origin xyz=0.0 -0.01 0.005 rpy=0 0.1 0 -> xyz=0.0 0.0 0.0 rpy=0 0.1 0
- joint camera_stick_joint: origin xyz=0.2735 0.01 0.005 rpy=0.0 0.0 0.0 -> xyz=-0.23199999999999998 0 0.069 rpy=0.0 0.0 0.0
- joint front_left_steering_joint: origin xyz=0.22050000000000003 0.1495 -0.029 rpy=0 0 0 -> xyz=0.1795 0.13 -0.069 rpy=0 0 0
- joint front_left_wheel_joint: limit effort=10.0 velocity=17.241379310344826 -> effort=10.0 velocity=17.391304347826086
- joint front_right_steering_joint: origin xyz=0.22050000000000003 -0.1495 -0.029 rpy=0 0 0 -> xyz=0.1795 -0.13 -0.069 rpy=0 0 0
- joint front_right_wheel_joint: limit effort=10.0 velocity=17.241379310344826 -> effort=10.0 velocity=17.391304347826086
- joint rear_left_wheel_joint: limit effort=10.0 velocity=17.241379310344826 -> effort=10.0 velocity=17.391304347826086; origin xyz=-0.22050000000000003 0.1495 -0.029 rpy=0 0 0 -> xyz=-0.1795 0.13 -0.069 rpy=0 0 0
- joint rear_right_wheel_joint: limit effort=10.0 velocity=17.241379310344826 -> effort=10.0 velocity=17.391304347826086; origin xyz=-0.22050000000000003 -0.1495 -0.029 rpy=0 0 0 -> xyz=-0.1795 -0.13 -0.069 rpy=0 0 0

File: robot_challenge_description/src/description/robot_challenge_description.xacro (robot description, xacro)
@@ -6,10 +6,11 @@
   -->
   <!-- Arguments -->
-  <xacro:arg name="body_length" default=".557" />
-  <xacro:arg name="body_width" default=".249" />
-  <xacro:arg name="body_height" default="0.241" />
+  <xacro:arg name="body_length" default=".474" />
+  <xacro:arg name="body_width" default=".192" />
+  <xacro:arg name="body_height" default="0.138" />
   <xacro:arg name="body_density" default="1000.0" />
-  <xacro:arg name="wheel_radius" default="0.058" />
-  <xacro:arg name="wheel_width" default="0.05" />
+  <xacro:arg name="wheel_radius" default="0.0575" />
+  <xacro:arg name="wheel_width" default="0.068" />
+  <xacro:arg name="wheel_base" default="0.275" />
   <xacro:arg name="wheel_density" default="1000.0" />
   <xacro:arg name="max_steering_angle" default="0.6108" />
@@ -20,5 +21,5 @@
   <xacro:arg name="camera_box_size" default="0.01" />
   <xacro:arg name="camera_stick_size" default="0.01" />
-  <xacro:arg name="camera_height" default=".01" />
+  <!-- <xacro:arg name="camera_height" default=".01" /> -->
   <xacro:arg name="camera_pitch" default="0.1" />
   <xacro:arg name="camera_fov" default="1.570796" />
@@ -26,4 +27,10 @@
   <xacro:arg name="image_width" default="640" />
   <xacro:arg name="image_height" default="480" />
+  <!-- <xacro:arg name="camera_length" default=".0254" />
+  <xacro:arg name="camera_width" default=".10" />
+  <xacro:arg name="camera_height" default="0.0254" />
+  <xacro:arg name="lidar_length" default=".10" />
+  <xacro:arg name="lidar_width" default=".10" />
+  <xacro:arg name="lidar_height" default="0.10" /> -->
   <!-- Mathematical Constants -->
   <xacro:property name="PI" value="3.14159265"/>
@@ -60,8 +67,29 @@
   <xacro:property name="wheel_inertia_z" value="${1.0/2.0 * wheel_mass * wheel_radius * wheel_radius}"/>
   <xacro:property name="max_wheel_angular_velocity" value="${max_velocity / wheel_radius}"/>
+  <xacro:property name="camera_length" value=".0254" />
+  <xacro:property name="camera_width" value=".10" />
+  <xacro:property name="camera_height" value="0.0254" />
+  <xacro:property name="lidar_radius" value=".0325" />
+  <xacro:property name="lidar_height" value="0.0528" />
   <!-- Macros -->
   <xacro:macro name="box_inertia" params="m x y z">
     <inertia ixx="${m*(y*y+z*z)/12}" ixy = "0" ixz = "0" iyy="${m*(x*x+z*z)/12}" iyz = "0" izz="${m*(x*x+z*z)/12}" />
   </xacro:macro>
+  <!-- Materials -->
+  <material name="gray_25">
+    <color rgba="0.25 0.25 0.25 1.0"/>
+  </material>
+  <material name="gray_50">
+    <color rgba="0.50 0.50 0.50 1.0"/>
+  </material>
+  <material name="gray_75">
+    <color rgba="0.75 0.75 0.75 1.0"/>
+  </material>
+  <material name="camera_color">
+    <color rgba="0.70 0.2 0.2 1.0"/>
+  </material>
+  <material name="lidar_color">
+    <color rgba="0.2 0.7 0.2 1.0"/>
+  </material>
   <!-- Links -->
   <!-- Body Link -->
@@ -72,7 +100,5 @@
         <box size="${body_length} ${body_width} ${body_height}"/>
       </geometry>
-      <material name="body_material">
-        <color rgba="0.25 0.25 0.25 1.0"/>
-      </material>
+      <material name="gray_25"/>
     </visual>
     <collision>
@@ -249,15 +275,13 @@
       <origin xyz="0 0 0" rpy="0 0 0"/>
       <geometry>
-        <box size="${camera_box_size} ${camera_box_size} ${camera_box_size}"/>
-      </geometry>
-    </collision>
-    <visual>
-      <origin xyz="0 0 0" rpy="0 0 0"/>
-      <geometry>
-        <box size="${camera_box_size} ${camera_box_size} ${camera_box_size}"/>
-      </geometry>
-      <material name="camera_material">
-        <color rgba="0.0 0.0 0.0 1.0"/>
-      </material>
+        <box size="${camera_length} ${camera_width} ${camera_height}"/>
+      </geometry>
+    </collision>
+    <visual>
+      <origin xyz="0 0 0" rpy="0 0 0"/>
+      <geometry>
+        <box size="${camera_length} ${camera_width} ${camera_height}"/>
+      </geometry>
+      <material name="camera_color" />
     </visual>
     <inertial>
@@ -266,23 +290,43 @@
       <inertia ixx="1e-6" ixy="0" ixz="0" iyy="1e-6" iyz="0" izz="1e-6" />
     </inertial>
+  </link>
+  <!-- Lidar Link -->
+  <link name="lidar_link">
+    <collision>
+      <origin xyz="0 0 0" rpy="0 0 0"/>
+      <geometry>
+        <cylinder radius="${lidar_radius}" length="${lidar_height}"/>
+      </geometry>
+    </collision>
+    <visual>
+      <origin xyz="0 0 0" rpy="0 0 0"/>
+      <geometry>
+        <cylinder radius="${lidar_radius}" length="${lidar_height}"/>
+      </geometry>
+      <material name="lidar_color"/>
+    </visual>
   </link>
   <!-- IMU Link -->
   <link name="imu_link">
-    <visual>
-      <geometry>
-        <box size="0.1 0.1 0.1"/>
-      </geometry>
-    </visual>
-    <collision>
-      <geometry>
-        <box size="0.1 0.1 0.1"/>
-      </geometry>
-    </collision>
+    <collision>
+      <origin xyz="0 0 0" rpy="0 0 0"/>
+      <geometry>
+        <box size="${camera_length} ${camera_width} ${camera_height}"/>
+      </geometry>
+    </collision>
+    <visual>
+      <origin xyz="0 0 0" rpy="0 0 0"/>
+      <geometry>
+        <box size="${camera_length} ${camera_width} ${camera_height}"/>
+      </geometry>
+    </visual>
     <xacro:box_inertia m="0.1" x="0.1" y="0.1" z="0.1"/>
+  </link>
+  <link name="steering_wheel_link">
   </link>
   <!-- Joints -->
   <!-- Front Left Steering Joint -->
   <joint name="front_left_steering_joint" type="revolute">
-    <origin xyz="${wheel_offset} ${wheel_separation/2} -${wheel_radius/2}" rpy="0 0 0"/>
+    <origin xyz="${wheel_offset} ${wheel_separation/2} -${body_height/2}" rpy="0 0 0"/>
     <parent link="base_link"/>
     <child link="front_left_steering_link"/>
@@ -302,5 +346,5 @@
   <!-- Front Right Steering Joint -->
   <joint name="front_right_steering_joint" type="revolute">
-    <origin xyz="${wheel_offset} ${-wheel_separation/2} -${wheel_radius/2}" rpy="0 0 0"/>
+    <origin xyz="${wheel_offset} ${-wheel_separation/2} -${body_height/2}" rpy="0 0 0"/>
     <parent link="base_link"/>
     <child link="front_right_steering_link"/>
@@ -320,5 +364,5 @@
   <!-- Rear Left Wheel Joint -->
   <joint name="rear_left_wheel_joint" type="continuous">
-    <origin xyz="-${wheel_offset} ${wheel_separation/2} -${wheel_radius/2}" rpy="0 0 0"/>
+    <origin xyz="-${wheel_offset} ${wheel_separation/2} -${body_height/2}" rpy="0 0 0"/>
     <parent link="base_link"/>
     <child link="rear_left_wheel_link"/>
@@ -329,5 +373,5 @@
   <!-- Rear Right Wheel Joint -->
   <joint name="rear_right_wheel_joint" type="continuous">
-    <origin xyz="-${wheel_offset} ${-wheel_separation/2} -${wheel_radius/2}" rpy="0 0 0"/>
+    <origin xyz="-${wheel_offset} ${-wheel_separation/2} -${body_height/2}" rpy="0 0 0"/>
     <parent link="base_link"/>
     <child link="rear_right_wheel_link"/>
@@ -339,5 +383,5 @@
   <joint name="camera_stick_joint" type="fixed">
     <axis xyz="0 1 0" />
-    <origin xyz="${body_length/2 - camera_stick_size/2} ${camera_box_size/2 + camera_stick_size/2} ${camera_height/2}" rpy="0.0 0.0 0.0"/>
+    <origin xyz="-${body_length/2 - camera_stick_size/2} 0 ${body_height/2}" rpy="0.0 0.0 0.0"/>
     <parent link="base_link"/>
     <child link="camera_stick_link"/>
@@ -346,8 +390,15 @@
   <joint name="camera_joint" type="fixed">
     <axis xyz="0 1 0" />
-    <origin xyz="0.0 ${-camera_box_size/2 - camera_stick_size/2} ${camera_height/2}" rpy="0 ${camera_pitch} 0"/>
+    <!-- <origin xyz="0.0 ${-camera_box_size/2 - camera_stick_size/2} ${camera_height/2}" rpy="0 ${camera_pitch} 0"/> -->
     <origin xyz="0.0 0.0 0.0" rpy="0 ${camera_pitch} 0"/>
     <parent link="camera_stick_link"/>
     <child link="camera_link"/>
+  </joint>
+  <!-- Lidar Joint -->
+  <joint name="lidar_joint" type="fixed">
+    <axis xyz="0 1 0"/>
+    <origin xyz="${body_length/2 - 0.015} 0 ${body_height/2 - lidar_height/2}" rpy="0.0 0.0 0.0"/>
+    <parent link="base_link"/>
+    <child link="lidar_link"/>
   </joint>
   <!-- IMU Joint -->
@@ -356,4 +407,9 @@
     <child link="imu_link"/>
     <origin xyz="0 0 0.01"/>
+  </joint>
+  <joint name="steering_wheel_joint" type="continuous">
+    <parent link="base_link"/>
+    <child link="steering_wheel_link"/>
+    <origin xyz="0 0 0.0"/>
   </joint>
   <!-- Gazebo Parameters -->
@@ -411,5 +467,5 @@
     </joint>
     <joint name="rear_right_wheel_joint">
-      <command_interface name="velocity">gazebo_ackermann_steering_vehicle
+      <command_interface name="velocity">
         <param name="min">${-max_wheel_angular_velocity}</param>
         <param name="max">${max_wheel_angular_velocity}</param>
@@ -418,4 +474,6 @@
       <state_interface name="velocity"/>
       <state_interface name="effort"/>
+    </joint>
+    <joint name="steering_wheel_joint">
     </joint>
   </ros2_control>
@@ -464,5 +522,5 @@
         <alwaysOn>true</alwaysOn>
         <updateRate>0.0</updateRate>
-        <cameraName>vehicle_front_camera</cameraName>
+        <cameraName>front_camera</cameraName>
         <frameName>camera_link</frameName>
         <hackBaseline>0.07</hackBaseline>
@@ -479,5 +537,5 @@
    <plugin filename="libgazebo_ros_imu_sensor.so" name="imu_plugin">
       <ros>
-        <namespace>/demo</namespace>
+        <namespace>/sensors</namespace>
         <remapping>~/out:=imu</remapping>
       </ros>
@@ -543,4 +601,48 @@
   </sensor>
 </gazebo>
+<gazebo reference="lidar_link">
+  <sensor name="lidar_sensor" type="ray">
+    <pose> 0 0 0 0 0 0 </pose>
+    <update_rate>10</update_rate>
+    <ray>
+      <scan>
+          <horizontal>
+              <samples>500</samples>
+              <resolution>1</resolution>
+              <min_angle>-3.142</min_angle>
+              <max_angle>3.142</max_angle>
+          </horizontal>
+          <vertical>
+              <samples>1</samples>
+              <resolution>1</resolution>
+              <min_angle>0</min_angle>
+              <max_angle>0</max_angle>
+          </vertical>
+      </scan>
+      <range>
+          <min>0.3</min>
+          <max>40.0</max>
+          <resolution>0.001</resolution>
+      </range>
+      <noise>
+          <type>gaussian</type>
+          <mean>0.0</mean>
+          <stddev>0.0</stddev>
+      </noise>
+    </ray>
+    <plugin name="gazebo_ros_laser_controller" filename="libgazebo_ros_ray_sensor.so">
+      <ros>
+        <namespace>/sensors</namespace>
+        <remapping>~/out:=scan</remapping>
+      </ros>
+      <frame_name>lidar_link</frame_name>
+      <output_type>sensor_msgs/LaserScan</output_type>
+      <topic>scan</topic>
+      <min_range>0.3</min_range>
+      <max_range>40.0</max_range>
+      <gaussian_noise>0.008</gaussian_noise>
+    </plugin>
+  </sensor>
+</gazebo>
 <gazebo>
   <plugin filename="libgazebo_ros_ackermann_drive.so" name="ackermann_plugin">
@@ -566,4 +668,5 @@
     <rear_right_joint>rear_right_wheel_joint</rear_right_joint>
     <rear_left_joint>rear_left_wheel_joint</rear_left_joint>
+    <steering_wheel_joint>steering_wheel_joint</steering_wheel_joint>
     <wheel_separation>${body_width}</wheel_separation>
     <!-- output -->

Commit message: Visualize the lidar

File: robot_challenge_description/src/description/robot_challenge_description.urdf (robot description, URDF)
Before this commit: robot ackermann_steering_vehicle, 12 links, 11 joints
Joints:
- joint lidar_joint: origin xyz=0.22199999999999998 0 0.042600000000000006 rpy=0.0 0.0 0.0 -> xyz=0.237 0 0.042600000000000006 rpy=0.0 0.0 0.0

File: robot_challenge_description/src/description/robot_challenge_description.xacro (robot description, xacro)
@@ -398,5 +398,5 @@
   <joint name="lidar_joint" type="fixed">
     <axis xyz="0 1 0"/>
-    <origin xyz="${body_length/2 - 0.015} 0 ${body_height/2 - lidar_height/2}" rpy="0.0 0.0 0.0"/>
+    <origin xyz="${body_length/2} 0 ${body_height/2 - lidar_height/2}" rpy="0.0 0.0 0.0"/>
     <parent link="base_link"/>
     <child link="lidar_link"/>
@@ -602,7 +602,8 @@
 </gazebo>
 <gazebo reference="lidar_link">
-  <sensor name="lidar_sensor" type="ray">
+  <sensor name="lidar_sensor" type="gpu_lidar">
     <pose> 0 0 0 0 0 0 </pose>
     <update_rate>10</update_rate>
+    <visualize>true</visualize>
     <ray>
       <scan>
@@ -642,4 +643,6 @@
       <max_range>40.0</max_range>
       <gaussian_noise>0.008</gaussian_noise>
+      <always_on>1</always_on>
+      <render_engine>ogre2</render_engine>
     </plugin>
   </sensor>
