Commit message: Update to gazebo fortress as the ackermann plugin doesn't seem to be compatible with classic

File: robot_challenge_description/src/description/robot_challenge_description.urdf (robot description, URDF)
Before this commit: robot ackermann_steering_vehicle, 12 links, 11 joints
Links:
- added link body_link; collision box size=0.474 0.192 0.138; visual box size=0.474 0.192 0.138
- link base_link: geometry 
- link steering_wheel_link: mass None -> 1e-5
Joints:
- added joint body_joint: type fixed, parent base_link, child body_link, origin xyz=0 0 0 rpy=0 0 0

File: robot_challenge_description/src/description/robot_challenge_description.xacro (robot description, xacro)
@@ -95,5 +95,5 @@
   <!-- Body Link -->
   <link name="base_link">
-    <visual>
+    <!-- <visual>
       <origin xyz="0.0 0.0 0.0" rpy="0.0 0.0 0.0"/>
       <geometry>
@@ -107,5 +107,21 @@
         <box size="${body_length} ${body_width} ${body_height}"/>
       </geometry>
-    </collision>
+    </collision> -->
+  </link>
+  <link name="body_link">
+      <visual>
+      <origin xyz="0.0 0.0 0.0" rpy="0.0 0.0 0.0"/>
+      <geometry>
+        <box size="${body_length} ${body_width} ${body_height}"/>
+      </geometry>
+      <material name="gray_75"/>
+    </visual>
+    <collision>
+      <origin xyz="0.0 0.0 0.0" rpy="0.0 0.0 0.0"/>
+      <geometry>
+        <box size="${body_length} ${body_width} ${body_height}"/>
+      </geometry>
+    </collision>
+    <xacro:box_inertia m="3000" x="${body_length}" y="${body_width}" z="${body_height}"/>
   </link>
   <!-- Front Left Wheel -->
@@ -324,6 +340,16 @@
   </link>
   <link name="steering_wheel_link">
+    <inertial>
+      <mass value="1e-5" />
+      <origin xyz="0 0 0" rpy="0 0 0"/>
+      <inertia ixx="1e-6" ixy="0" ixz="0" iyy="1e-6" iyz="0" izz="1e-6" />
+    </inertial>
   </link>
   <!-- Joints -->
+  <joint name="body_joint" type="fixed">
+    <origin xyz="0 0 0" rpy="0 0 0"/>
+    <parent link="base_link"/>
+    <child link="body_link"/>
+  </joint>
   <!-- Front Left Steering Joint -->
   <joint name="front_left_steering_joint" type="revolute">
@@ -419,5 +445,5 @@
   </gazebo>
   <gazebo reference="front_right_wheel_link">
-    <mu1>100.0</mu1>gazebo_ackermann_steering_vehicle
+    <mu1>100.0</mu1>
     <mu2>100.0</mu2>
   </gazebo>
@@ -435,5 +461,5 @@
   </gazebo>
   <!-- Gazebo Control -->
-  <ros2_control name="control" type="system">
+  <ros2_control name="GazeboSimSystem" type="system">
     <hardware>
       <plugin>gz_ros2_control/GazeboSimSystem</plugin>
@@ -480,5 +506,5 @@
   <!-- Gazebo Plugins -->
   <gazebo>
-    <plugin filename="libgazebo_ros_joint_state_publisher.so" name="gz::sim::systems::JointStatePublisher">
+    <!-- <plugin filename="libgazebo_ros_joint_state_publisher.so" name="gz::sim::systems::JointStatePublisher">
       <topic>joint_states</topic>
       <joint_name>front_left_steering_joint</joint_name>
@@ -488,6 +514,31 @@
       <joint_name>rear_left_wheel_joint</joint_name>
       <joint_name>rear_right_wheel_joint</joint_name>
+    </plugin> -->
+    <plugin
+      filename="libignition-gazebo-ackermann-steering-system"
+      name="ignition::gazebo::systems::AckermannSteering">
+      <left_joint>front_left_wheel_joint</left_joint>
+      <left_joint>rear_left_wheel_joint</left_joint>
+      <right_joint>front_right_wheel_joint</right_joint>
+      <right_joint>rear_right_wheel_joint</right_joint>
+      <left_steering_joint>front_left_steering_joint</left_steering_joint>
+      <right_steering_joint>front_right_steering_joint</right_steering_joint>
+      <kingpin_width>1.0</kingpin_width>
+      <steering_limit>0.5</steering_limit>
+      <wheel_base>1.0</wheel_base>
+      <wheel_separation>1.25</wheel_separation>
+      <wheel_radius>0.3</wheel_radius>
+      <min_velocity>-1</min_velocity>
+      <max_velocity>1</max_velocity>
+      <min_acceleration>-3</min_acceleration>
+      <max_acceleration>3</max_acceleration>
+      <topic>cmd_vel</topic>
     </plugin>
-    <plugin filename="libgz_ros2_control-system.so" name="gz_ros2_control::GazeboSimROS2ControlPlugin">
+    <plugin filename="libignition-gazebo-joint-state-publisher-system.so"
+      name="ignition::gazebo::systems::JointStatePublisher">
+      <topic>joint_states</topic>
+      <update_rate>100</update_rate>
+    </plugin>
+    <plugin filename="gz_ros2_control-system" name="gz_ros2_control::GazeboSimROS2ControlPlugin">
       <parameters>$(find robot_challenge_description)/config/gz_ros2_control.yaml</parameters>
     </plugin>
@@ -498,5 +549,5 @@
   <!-- Camera -->
   <gazebo reference="camera_link">
-    <sensor type="camera" name="vehicle_front_camera">
+    <sensor name="vehicle_front_camera" type="camera">
       <update_rate>${camera_fps}</update_rate>
       <visualize>true</visualize>
@@ -519,5 +570,5 @@
         </noise>
       </camera>
-      <plugin name="camera_controller" filename="libgazebo_ros_camera.so">
+      <!-- <plugin name="camera_controller" filename="libgazebo_ros_camera.so">
         <alwaysOn>true</alwaysOn>
         <updateRate>0.0</updateRate>
@@ -530,16 +581,9 @@
         <distortionT1>0.0</distortionT1>
         <distortionT2>0.0</distortionT2>
-      </plugin>
+      </plugin> -->
     </sensor>
   </gazebo>
  <gazebo reference="imu_link">
   <sensor name="imu_sensor" type="imu">
-   <plugin filename="libgazebo_ros_imu_sensor.so" name="imu_plugin">
-      <ros>
-        <namespace>/sensors</namespace>
-        <remapping>~/out:=imu</remapping>
-      </ros>
-      <initial_orientation_as_reference>false</initial_orientation_as_reference>
-    </plugin>
     <always_on>true</always_on>
     <update_rate>100</update_rate>
@@ -605,4 +649,6 @@
     <pose> 0 0 0 0 0 0 </pose>
     <update_rate>10</update_rate>
+    <topic>LaserScan</topic>
+    <always_on>1</always_on>
     <visualize>true</visualize>
     <ray>
@@ -632,53 +678,5 @@
       </noise>
     </ray>
-    <plugin name="gazebo_ros_laser_controller" filename="libgazebo_ros_ray_sensor.so">
-      <ros>
-        <namespace>/sensors</namespace>
-        <remapping>~/out:=scan</remapping>
-      </ros>
-      <frame_name>lidar_link</frame_name>
-      <output_type>sensor_msgs/LaserScan</output_type>
-      <topic>scan</topic>
-      <min_range>0.3</min_range>
-      <max_range>40.0</max_range>
-      <gaussian_noise>0.008</gaussian_noise>
-      <always_on>1</always_on>
-      <render_engine>ogre2</render_engine>
-    </plugin>
   </sensor>
 </gazebo>
-<gazebo>
-  <plugin filename="libgazebo_ros_ackermann_drive.so" name="ackermann_plugin">
-    <ros>
-      <namespace>ackermann</namespace>
-      <remapping>cmd_vel:=cmd_vel</remapping>
-      <remapping>odom:=odom</remapping>
-      <remapping>distance:=distance</remapping>
-    </ros>
-    <!-- <left_joint>front_left_wheel_joint</left_joint>
-    <left_joint>rear_left_wheel_joint</left_joint>
-    <right_joint>front_right_wheel_joint</right_joint>
-    <right_joint>rear_right_wheel_joint</right_joint>
-    -->
-    <!--
-    Docs
-    https://docs.ros.org/en/rolling/p/gazebo_plugins/generated/classgazebo__plugins_1_1GazeboRosAckermannDrive.html
-    -->
-    <left_steering_joint>front_left_steering_joint</left_steering_joint>
-    <right_steering_joint>front_right_steering_joint</right_steering_joint>
-    <front_right_joint>front_right_wheel_joint</front_right_joint>
-    <front_left_joint>front_left_wheel_joint</front_left_joint>
-    <rear_right_joint>rear_right_wheel_joint</rear_right_joint>
-    <rear_left_joint>rear_left_wheel_joint</rear_left_joint>
-    <steering_wheel_joint>steering_wheel_joint</steering_wheel_joint>
-    <wheel_separation>${body_width}</wheel_separation>
-    <!-- output -->
-    <publish_odom>true</publish_odom>
-    <publish_odom_tf>true</publish_odom_tf>
-    <publish_wheel_tf>true</publish_wheel_tf>
-    <publish_distance>true</publish_distance>
-    <odometry_frame>odom_demo</odometry_frame>
-    <robot_base_frame>base_link</robot_base_frame>
-  </plugin>
-</gazebo>
 </robot>
